File: DC Offset.brd (EAGLE design)
At the start: 18.3 x 100 mm, 21 parts, among them IC1 TL072D

Commit message: Reinstall
Parts:
- added R7: 10k, GMSN:R0805
- added R8: 1k, GMSN:R0805
- R1, R2, R3, R4, R5, R6: value 100k -> 10k
Connections:
- removed net N$10: IC1.6, IC1.7
- removed net N$8: IC1.2, R1.2, R6.1
- new net N$2: IC1.7, R7.2, R8.1
- new net N$3: OUT.TIP, R8.2
- new net N$4: IC1.6, R1.2, R7.1
- net GND: now also IC1.3; no longer R1.1
- net N$6: now also IC1.2, R6.1; no longer IC1.3
- net N$9: now also R1.1; no longer OUT.TIP
Routing:
- net N$8: track 7.66 -> 0.00 mm
- net N$6: track 27.4 -> 29.8 mm
- net N$10: track 1.27 -> 0.00 mm
