File: DC Offset.sch (EAGLE design)
At the start: 19 parts, among them IC1 TL072D

Commit message: Reinstall
Parts:
- added R7: 10k, GMSN:R-US_R0805
- added R8: 1k, GMSN:R-US_R0805
- R1, R2, R3, R4, R5, R6: value 100k -> 10k
Connections:
- removed net N$10: IC1B.-IN, IC1B.OUT
- removed net N$8: IC1A.-IN, R1.2, R6.1
- new net N$2: IC1B.OUT, R7.2, R8.1
- new net N$3: OUT.TIP, R8.2
- new net N$4: IC1B.-IN, R1.2, R7.1
- net GND: now also IC1A.+IN; no longer R1.1
- net N$6: now also IC1A.-IN, R6.1; no longer IC1A.+IN
- net N$9: now also R1.1; no longer OUT.TIP
Other:
- moved on the sheet: IC1B, OUT, R1
